Commit message: Black-Box Mode

File: mir_description/urdf/include/mir_100_v1.urdf.xacro (robot description, xacro)
@@ -154,5 +154,5 @@
       <parent link="${prefix}base_link" />
       <child link="${prefix}imu_link" />
-      <origin xyz="0.0 0.0 0.25" rpy="0 0 0" />  <!-- same as real MiR -->
+      <origin xyz="0.0 0.0 0.25" rpy="0 0 1.570789" />  <!-- same as real MiR -->
     </joint>
     <link name="${prefix}imu_link" />
